Commit message: code cleanup and commenting, readme to finish

File: robot_control/urdf/robot4.xacro (robot description, xacro)
@@ -140,13 +140,13 @@
   <link name = "camera_stick">
     <collision>
-      <origin xyz = "0 0 ${stick_height/2}" rpy="0 0 0"/>
+      <origin xyz = "0 0 0.1" rpy="0 0 0"/>
       <geometry>
-        <box size = "0.05 0.05 0.2"/>
+        <box size = "0.05 0.05 0.1"/>
       </geometry>
     </collision>
     <visual>
-      <origin xyz = "0 0 ${stick_height/2}" rpy="0 0 0"/>
+      <origin xyz = "0 0 0.1" rpy="0 0 0"/>
       <geometry>
-        <box size = "0.05 0.05 ${stick_height}"/>
+        <box size = "0.05 0.05 0.1"/>
       </geometry>
       <material name="orange"/>
@@ -166,5 +166,5 @@
   <joint name="camera_joint" type="continuous">
     <axis xyz="0 0 1" />
-    <origin xyz="0 0 ${stick_height/2}" rpy="0 0 0"/>
+    <origin xyz="0 0 0.1" rpy="0 0 0"/>
     <parent link="camera_stick"/>
     <child link="camera_link"/>
